File: hardware/HeikouBoxCore/HeikouBoxCore.sch (KiCad schematic (older format))
At the start: 28 parts, among them U1 EP3C25E144

Commit message: Update to local libraries, minor work
Parts:
- A1: footprint KasaneK-Custom-Parts:HeikouBox-Core-Top -> ksk-heikoubox:HeikouBox-Core-Top; symbol KasaneK-Custom-Parts:HeikouBox-Core -> ksk-heikoubox:HeikouBox-Core
- U1: footprint KasaneK-Custom-Parts:EQFP-144-HANDSOLDER -> ksk-heikoubox:EQFP-144-HANDSOLDER; symbol KasaneK-Custom-Parts:EP3C25E144 -> ksk-heikoubox:EP3C25E144
Changed lines of the file:
@@
 EESchema Schematic File Version 4
-LIBS:HeikouBoxCore-cache
-EELAYER 26 0
+EELAYER 30 0
 EELAYER END
 $Descr A4 11693 8268
@@
 $EndDescr
 $Comp
-L KasaneK-Custom-Parts:EP3C25E144 U1
+L ksk-heikoubox:EP3C25E144 U1
 U 1 1 5E5BAA29
 P 900 700
 F 0 "U1" H 1200 865 50  0000 C CNN
 F 1 "EP3C25E144" H 1200 774 50  0000 C CNN
-F 2 "KasaneK-Custom-Parts:EQFP-144-HANDSOLDER" H 3350 550 50  0001 C CNN
+F 2 "ksk-heikoubox:EQFP-144-HANDSOLDER" H 3350 550 50  0001 C CNN
 F 3 "" H 650 2900 50  0001 C CNN
 	1    900  700
@@
 $EndComp
 $Comp
-L KasaneK-Custom-Parts:EP3C25E144 U1
+L ksk-heikoubox:EP3C25E144 U1
 U 2 1 5E5BAA8C
 P 2250 700
 F 0 "U1" H 2725 865 50  0000 C CNN
 F 1 "EP3C25E144" H 2725 774 50  0000 C CNN
-F 2 "KasaneK-Custom-Parts:EQFP-144-HANDSOLDER" H 4700 550 50  0001 C CNN
+F 2 "ksk-heikoubox:EQFP-144-HANDSOLDER" H 4700 550 50  0001 C CNN
 F 3 "" H 2000 2900 50  0001 C CNN
 	2    2250 700
@@
 $EndComp
 $Comp
-L KasaneK-Custom-Parts:EP3C25E144 U1
+L ksk-heikoubox:EP3C25E144 U1
 U 3 1 5E5BAB2D
 P 3750 700
 F 0 "U1" H 4131 865 50  0000 C CNN
 F 1 "EP3C25E144" H 4131 774 50  0000 C CNN
-F 2 "KasaneK-Custom-Parts:EQFP-144-HANDSOLDER" H 6200 550 50  0001 C CNN
+F 2 "ksk-heikoubox:EQFP-144-HANDSOLDER" H 6200 550 50  0001 C CNN
 F 3 "" H 3500 2900 50  0001 C CNN
 	3    3750 700
@@
 	4400 1800 4400 1900
 $Comp
-L KasaneK-Custom-Parts:HeikouBox-Core A1
+L ksk-heikoubox:HeikouBox-Core A1
 U 1 1 5EF5786F
 P 850 5250
 F 0 "A1" H 1250 5415 50  0000 C CNN
 F 1 "HeikouBox-Core" H 1250 5324 50  0000 C CNN
-F 2 "KasaneK-Custom-Parts:HeikouBox-Core-Top" H 1150 5250 50  0001 C CNN
+F 2 "ksk-heikoubox:HeikouBox-Core-Top" H 1150 5250 50  0001 C CNN
 F 3 "" H 1150 5250 50  0001 C CNN
 	1    850  5250
@@
 $EndComp
 $Comp
-L KasaneK-Custom-Parts:HeikouBox-Core A1
+L ksk-heikoubox:HeikouBox-Core A1
 U 2 1 5EF57BDC
 P 2350 5250
 F 0 "A1" H 2750 5415 50  0000 C CNN
 F 1 "HeikouBox-Core" H 2750 5324 50  0000 C CNN
-F 2 "KasaneK-Custom-Parts:HeikouBox-Core-Top" H 2650 5250 50  0001 C CNN
+F 2 "ksk-heikoubox:HeikouBox-Core-Top" H 2650 5250 50  0001 C CNN
 F 3 "" H 2650 5250 50  0001 C CNN
 	2    2350 5250
@@
 $EndComp
 $Comp
-L KasaneK-Custom-Parts:HeikouBox-Core A1
+L ksk-heikoubox:HeikouBox-Core A1
 U 3 1 5EF57CAD
 P 3850 5250
 F 0 "A1" H 4250 5415 50  0000 C CNN
 F 1 "HeikouBox-Core" H 4250 5324 50  0000 C CNN
-F 2 "KasaneK-Custom-Parts:HeikouBox-Core-Top" H 4150 5250 50  0001 C CNN
+F 2 "ksk-heikoubox:HeikouBox-Core-Top" H 4150 5250 50  0001 C CNN
 F 3 "" H 4150 5250 50  0001 C CNN
 	3    3850 5250
@@
 $EndComp
 $Comp
-L KasaneK-Custom-Parts:HeikouBox-Core A1
+L ksk-heikoubox:HeikouBox-Core A1
 U 4 1 5EF57D70
 P 5350 5250
 F 0 "A1" H 5750 5415 50  0000 C CNN
 F 1 "HeikouBox-Core" H 5750 5324 50  0000 C CNN
-F 2 "KasaneK-Custom-Parts:HeikouBox-Core-Top" H 5650 5250 50  0001 C CNN
+F 2 "ksk-heikoubox:HeikouBox-Core-Top" H 5650 5250 50  0001 C CNN
 F 3 "" H 5650 5250 50  0001 C CNN
 	4    5350 5250

Commit message: Okay let's do this properly
Parts:
- added MH1, MH2, MH3, MH4: M3, MountingHole:MountingHole_3.2mm_M3, symbol Mechanical:MountingHole
- J1: renamed from A1; value HeikouBox-Core -> L; footprint ksk-heikoubox:HeikouBox-Core-Top -> KSK_HeikouBox:PinHeader_2x12_P2.00mm_Vertical-MIRRORED; symbol ksk-heikoubox:HeikouBox-Core -> KSK_HeikouBox:HeikouBox_Core_Conn_Left
- J2: renamed from A1; value HeikouBox-Core -> B; footprint ksk-heikoubox:HeikouBox-Core-Top -> KSK_HeikouBox:PinHeader_2x12_P2.00mm_Vertical-MIRRORED; symbol ksk-heikoubox:HeikouBox-Core -> KSK_HeikouBox:HeikouBox_Core_Conn_Bottom
- J3: renamed from A1; value HeikouBox-Core -> R; footprint ksk-heikoubox:HeikouBox-Core-Top -> KSK_HeikouBox:PinHeader_2x12_P2.00mm_Vertical-MIRRORED; symbol ksk-heikoubox:HeikouBox-Core -> KSK_HeikouBox:HeikouBox_Core_Conn_Right
- J4: renamed from A1; value HeikouBox-Core -> T; footprint ksk-heikoubox:HeikouBox-Core-Top -> KSK_HeikouBox:PinHeader_2x12_P2.00mm_Vertical-MIRRORED; symbol ksk-heikoubox:HeikouBox-Core -> KSK_HeikouBox:HeikouBox_Core_Conn_Top
- U1: footprint ksk-heikoubox:EQFP-144-HANDSOLDER -> KSK_HeikouBox:EQFP-144-HANDSOLDER; symbol ksk-heikoubox:EP3C25E144 -> KSK_HeikouBox:EP3C25E144
Connections:
- net A11: now also J3.7 (A11); no longer J3.55 (A11)
- net A4: now also J4.18 (A4); no longer J4.42 (A4)
- net A5: now also J4.20 (A5); no longer J4.44 (A5)
- net A6: now also J4.22 (A6); no longer J4.46 (A6)
- net A7: now also J4.24 (A7); no longer J4.48 (A7)
- net A8: now also J3.5 (A8); no longer J3.53 (A8)
- net A9: now also J3.3 (A9); no longer J3.51 (A9)
- net BLU0: now also J2.7 (BLU0); no longer J2.79 (BLU0)
- net BLU1: now also J2.9 (BLU1); no longer J2.81 (BLU1)
- net BLU2: now also J2.8 (BLU2); no longer J2.80 (BLU2)
- net BLU3: now also J2.5 (BLU3); no longer J2.77 (BLU3)
- net BLU4: now also J2.3 (BLU4); no longer J2.75 (BLU4)
- net CAS: now also J4.2 (CAS); no longer J4.26 (CAS)
- net CFGDONE: now also J3.10 (CFGDONE); no longer J3.58 (CFGDONE)
- net CLK: now also J3.8 (CLK); no longer J3.56 (CLK)
- net CLK14: now also J2.13 (CLK14); no longer J2.85 (CLK14)
- net CLK28: now also J4.14 (CLK28); no longer J4.38 (CLK28)
- net D0: now also J4.16 (D0); no longer J4.40 (D0)
- net D1: now also J4.15 (D1); no longer J4.39 (D1)
- net D10: now also J3.4 (D10); no longer J3.52 (D10)
- net D11: now also J3.6 (D11); no longer J3.54 (D11)
- net D12: now also J4.23 (D12); no longer J4.47 (D12)
- net D13: now also J4.21 (D13); no longer J4.45 (D13)
- net D14: now also J4.19 (D14); no longer J4.43 (D14)
- net D15: now also J4.17 (D15); no longer J4.41 (D15)
- net D2: now also J4.10 (D2); no longer J4.34 (D2)
- net D3: now also J4.9 (D3); no longer J4.33 (D3)
- net D4: now also J4.8 (D4); no longer J4.32 (D4)
- net D5: now also J4.7 (D5); no longer J4.31 (D5)
- net D6: now also J4.6 (D6); no longer J4.30 (D6)
- net D7: now also J4.5 (D7); no longer J4.29 (D7)
- net D8: now also J3.15 (D8); no longer J3.63 (D8)
- net D9: now also J3.2 (D9); no longer J3.50 (D9)
- net GND: now also J3.1 (GND), J3.24 (GND); no longer J3.49 (GND), J3.72 (GND)
- net GRN0: now also J2.24 (GRN0); no longer J2.96 (GRN0)
- net GRN1: now also J2.22 (GRN1); no longer J2.94 (GRN1)
- net GRN2: now also J2.20 (GRN2); no longer J2.92 (GRN2)
- net GRN3: now also J2.18 (GRN3); no longer J2.90 (GRN3)
- net GRN4: now also J2.17 (GRN4); no longer J2.89 (GRN4)
- net GRN5: now also J2.15 (GRN5); no longer J2.87 (GRN5)
- net LDQM: now also J4.4 (LDQM); no longer J4.28 (LDQM)
- net MDB5: now also J4.13 (MDB5); no longer J4.37 (MDB5)
- net MDB6: now also J4.12 (MDB6); no longer J4.36 (MDB6)
- net MDB7: now also J4.11 (MDB7); no longer J4.35 (MDB7)
- net NVSYNC: now also J2.2 (NVSYNC); no longer J2.74 (NVSYNC)
- net RED0: now also J3.16 (RED0); no longer J3.64 (RED0)
- net RED1: now also J3.17 (RED1); no longer J3.65 (RED1)
- net RED2: now also J3.18 (RED2); no longer J3.66 (RED2)
- net RED3: now also J3.19 (RED3); no longer J3.67 (RED3)
- net RED4: now also J3.21 (RED4); no longer J3.69 (RED4)
- net UDQM: now also J3.9 (UDQM); no longer J3.57 (UDQM)
- net V12: now also J3.23 (V12); no longer J3.71 (V12)
- net V25: now also J4.1 (V25); no longer J4.25 (V25)
- net V33: now also J2.1 (V33); no longer J2.73 (V33)
- net VID0: now also J3.11 (VID0); no longer J3.59 (VID0)
- net VID1: now also J3.12 (VID1); no longer J3.60 (VID1)
- net VID10: now also J2.14 (VID10); no longer J2.86 (VID10)
- net VID11: now also J2.12 (VID11); no longer J2.84 (VID11)
- net VID12: now also J2.11 (VID12); no longer J2.83 (VID12)
- net VID13: now also J2.10 (VID13); no longer J2.82 (VID13)
- net VID14: now also J2.6 (VID14); no longer J2.78 (VID14)
- net VID15: now also J2.4 (VID15); no longer J2.76 (VID15)
- net VID2: now also J3.13 (VID2); no longer J3.61 (VID2)
- net VID3: now also J3.14 (VID3); no longer J3.62 (VID3)
- net VID4: now also J3.20 (VID4); no longer J3.68 (VID4)
- net VID5: now also J3.22 (VID5); no longer J3.70 (VID5)
- net VID6: now also J2.23 (VID6); no longer J2.95 (VID6)
- net VID7: now also J2.21 (VID7); no longer J2.93 (VID7)
- net VID8: now also J2.19 (VID8); no longer J2.91 (VID8)
- net VID9: now also J2.16 (VID9); no longer J2.88 (VID9)
- net WE: now also J4.3 (WE); no longer J4.27 (WE)
