File: hardware/HeikouBox/HeikouBox.sch (KiCad schematic (older format))
At the start: 4 parts

Commit message: Mainboard v0.1 PCB ready for export
Changed lines of the file:
@@
 $EndSheet
 Wire Bus Line
-	1900 2250 3550 2250
+	1900 2250 3600 2250
 $Comp
 L Mechanical:MountingHole MH1
@@
 	1900 2100 2800 2100
 Wire Wire Line
-	1900 2300 3550 2300
-Wire Wire Line
-	3550 2350 1900 2350
-Wire Wire Line
-	1900 2400 3550 2400
-Wire Wire Line
-	1900 2450 3550 2450
+	1900 2300 3600 2300
+Wire Wire Line
+	3600 2350 1900 2350
+Wire Wire Line
+	1900 2400 3600 2400
+Wire Wire Line
+	1900 2450 3600 2450
 $Sheet
 S 2100 1000 550  600
@@
 F0 "part3-av" 25
 F1 "part3-av.sch" 25
-F2 "5V" I L 2100 1050 25
-F3 "GND" I L 2100 1150 25
-F4 "RED[0..4]" I L 2100 1250 25
-F5 "GRN[0..5]" I L 2100 1300 25
-F6 "BLU[0..4]" I L 2100 1350 25
-F7 "NHSYNC" I L 2100 1400 25
-F8 "NVSYNC" I L 2100 1450 25
-F9 "LSIGMA" I L 2100 1500 25
-F10 "RSIGMA" I L 2100 1550 25
-F11 "3V3" I L 2100 1100 25
-$EndSheet
-Wire Wire Line
-	2050 1050 2100 1050
-Wire Wire Line
-	2100 1100 2000 1100
-Wire Wire Line
-	4150 1050 4100 1050
-Wire Wire Line
-	3450 1100 3550 1100
-Wire Wire Line
-	3550 1150 3400 1150
+F2 "GND" I L 2100 1100 25
+F3 "RED[0..4]" I L 2100 1250 25
+F4 "GRN[0..5]" I L 2100 1300 25
+F5 "BLU[0..4]" I L 2100 1350 25
+F6 "NHSYNC" I L 2100 1400 25
+F7 "NVSYNC" I L 2100 1450 25
+F8 "LSIGMA" I L 2100 1500 25
+F9 "RSIGMA" I L 2100 1550 25
+F10 "3V3" I L 2100 1050 25
+$EndSheet
+Wire Wire Line
+	2100 1050 2000 1050
+Wire Wire Line
+	3450 1150 3600 1150
+Wire Wire Line
+	3600 1200 3400 1200
 Wire Wire Line
 	2800 1050 2750 1050
@@
 3
 Wire Wire Line
-	3550 1250 3350 1250
-Wire Wire Line
-	3550 1300 3350 1300
-Wire Wire Line
-	3550 1350 3350 1350
-Wire Wire Line
-	3550 1400 3350 1400
-Wire Wire Line
-	3350 1450 3550 1450
-Wire Wire Line
-	3350 1500 3550 1500
-Wire Wire Line
-	4150 600  4150 1050
-Wire Wire Line
-	2050 1050 2050 700
-Wire Wire Line
-	3450 750  3450 1100
+	3450 750  3450 1150
 Wire Wire Line
 	2750 750  3450 750
@@
 	1200 850  1200 1150
 Wire Wire Line
-	3400 900  3400 1150
+	3400 900  3400 1200
 Wire Wire Line
 	2700 900  2700 1100
@@
 	1100 900  1150 900
 Wire Wire Line
-	1100 600  4150 600
-Wire Wire Line
-	1100 700  2050 700
-Wire Wire Line
-	2100 1150 1950 1150
-Wire Wire Line
 	1150 900  1950 900
 Wire Wire Line
 	1300 750  2000 750
-Wire Wire Line
-	2000 1100 2000 750
 Connection ~ 2000 750
 Wire Wire Line
 	2000 750  2750 750
-Wire Wire Line
-	1950 1150 1950 900
 Connection ~ 1950 900
 Wire Wire Line
 	1950 900  2700 900
-$Sheet
-S 3550 1000 550  1500
-U 646E3FCF
-F0 "part5-hub" 25
-F1 "part5-hub.sch" 25
-F2 "VUSB" O R 4100 1050 25
-F3 "GND" I L 3550 1150 25
-F4 "3V3" I L 3550 1100 25
-F5 "cfg_NCFG" O L 3550 2300 25
-F6 "cfg_NSTAT" I L 3550 2400 25
-F7 "cfg_DCLK" O L 3550 2350 25
-F8 "mdb[0..7]" B L 3550 2250 25
-F9 "mem_XWE" O L 3550 1450 25
-F10 "mem_XCAS" O L 3550 1400 25
-F11 "mem_CKE" O L 3550 1250 25
-F12 "mem_XCLK" O L 3550 1300 25
-F13 "mem_XRAS" O L 3550 1350 25
-F14 "mem_XAP" O L 3550 1500 25
-F15 "cfg_DONE" I L 3550 2450 25
-F16 "5V" I L 3550 1050 25
-$EndSheet
 $Sheet
 S 2800 1000 550  1150
@@
 F11 "CAS" I L 2800 2050 25
 F12 "RAS" I L 2800 2000 25
-F13 "CKE" I R 3350 1250 25
-F14 "XCAS" I R 3350 1400 25
-F15 "XWE" I R 3350 1450 25
-F16 "XAP" I R 3350 1500 25
-F17 "XCLK" I R 3350 1300 25
-F18 "XRAS" I R 3350 1350 25
 $EndSheet
 $Sheet
@@
 $EndSheet
 Wire Wire Line
-	3550 1050 3500 1050
-Wire Wire Line
-	3500 1050 3500 700
-Wire Wire Line
-	3500 700  2050 700
-Connection ~ 2050 700
+	3600 1100 3500 1100
+Wire Wire Line
+	1100 700  3500 700
+$Sheet
+S 3600 1000 550  1500
+U 646E3FCF
+F0 "part5-hub" 25
+F1 "part5-hub.sch" 25
+F2 "VUSB" B L 3600 1050 25
+F3 "GND" B L 3600 1200 25
+F4 "3V3" I L 3600 1150 25
+F5 "cfg_NCFG" O L 3600 2300 25
+F6 "cfg_NSTAT" I L 3600 2400 25
+F7 "cfg_DCLK" O L 3600 2350 25
+F8 "mdb[0..7]" B L 3600 2250 25
+F9 "cfg_DONE" I L 3600 2450 25
+F10 "5V" I L 3600 1100 25
+$EndSheet
+Wire Wire Line
+	1100 600  3550 600
+Wire Wire Line
+	3500 1100 3500 700
+Wire Wire Line
+	3550 600  3550 1050
+Wire Wire Line
+	3600 1050 3550 1050
+Wire Wire Line
+	1950 1100 1950 900
+Wire Wire Line
+	2000 1050 2000 750
+Wire Wire Line
+	1950 1100 2100 1100
 $EndSCHEMATC

Commit message: Tidy up power nets
Changed lines of the file:
@@
 F12 "RAS" I L 2800 2000 25
-$EndSheet
-$Sheet
-S 550  550  550  400
-U 644CBAED
-F0 "part1-power" 25
-F1 "part1-power.sch" 25
-F2 "5V" O R 1100 700 25
-F3 "VUSB" I R 1100 600 25
-F4 "GND" O R 1100 900 25
-F5 "3V3" O R 1100 750 25
-F6 "2V5" O R 1100 800 25
-F7 "1V2" O R 1100 850 25
 $EndSheet
 Wire Wire Line
@@
 F1 "part5-hub.sch" 25
 F2 "VUSB" B L 3600 1050 25
-F3 "GND" B L 3600 1200 25
+F3 "GND" I L 3600 1200 25
 F4 "3V3" I L 3600 1150 25
 F5 "cfg_NCFG" O L 3600 2300 25
@@
 Wire Wire Line
 	1950 1100 2100 1100
+$Sheet
+S 550  550  550  400
+U 644CBAED
+F0 "part1-power" 25
+F1 "part1-power.sch" 25
+F2 "5V" O R 1100 700 25
+F3 "VUSB" B R 1100 600 25
+F4 "GND" O R 1100 900 25
+F5 "3V3" O R 1100 750 25
+F6 "2V5" O R 1100 800 25
+F7 "1V2" O R 1100 850 25
+$EndSheet
 $EndSCHEMATC
