File: hardware/HeikouBox/part1-power.sch (KiCad schematic (older format))
At the start: 11 parts, among them U101 LD1117S33TR, U102 LD1117S25TR, U103 LD1117S12TR

Commit message: Mostly routed board
Parts:
- added J101: 5V, KSK_HeikouBox:BarrelJack_Multi, symbol Connector:Barrel_Jack_Switch
- added JP101: Power, Connector_PinHeader_2.54mm:PinHeader_1x03_P2.54mm_Vertical, symbol Jumper:Jumper_3_Bridged12
- C101, C104, C105, C106: footprint Capacitor_SMD:C_0603_1608Metric_Pad1.05x0.95mm_HandSolder -> Capacitor_SMD:C_1206_3216Metric_Pad1.33x1.80mm_HandSolder; symbol Device:C -> Device:CP1
- C102: footprint Capacitor_SMD:C_0603_1608Metric_Pad1.05x0.95mm_HandSolder -> Capacitor_SMD:C_0603_1608Metric_Pad1.08x0.95mm_HandSolder
- F101: value Poly 0.5A -> Poly 1A
- R101: footprint Resistor_SMD:R_0603_1608Metric_Pad1.05x0.95mm_HandSolder -> Resistor_SMD:R_0603_1608Metric_Pad0.98x0.95mm_HandSolder
Connections:
- net GND: now also J101.2
- net VUSB: now also JP101.3 (B); no longer F101.2
- new net: J101.1, JP101.1 (A)
- new net: F101.2, JP101.2 (C)
- no-connect marks 0 -> 1
Other:
- moved on the sheet: C102, D101, F101, R101, U101, U102, U103

Commit message: Mainboard v0.1 PCB ready for export
Parts:
- removed JP101: Power, Connector_PinHeader_2.54mm:PinHeader_1x03_P2.54mm_Vertical, symbol Jumper:Jumper_3_Bridged12
- added D102: D, Diode_SMD:D_SOD-123, symbol Device:D
- added D103: 5.6V, Diode_SMD:D_SOD-123, symbol Device:D_Zener
- added F102: Poly 200mA, Fuse:Fuse_0805_2012Metric_Pad1.15x1.40mm_HandSolder, symbol Device:Polyfuse_Small
- F101: value Poly 1A -> Poly 2A; footprint Fuse:Fuse_0805_2012Metric_Pad1.15x1.40mm_HandSolder -> Fuse:Fuse_1206_3216Metric_Pad1.42x1.75mm_HandSolder
- R101: value 1K -> 330R
Connections:
- net 3V3: now also D101.2 (A)
- net 5V: now also F101.2, D103.1 (K), F102.1; no longer D101.2 (A), F101.1
- net GND: now also D103.2 (A)
- net VUSB: now also D102.1 (K)
- net at J101.1: now also F101.1
- new net: D102.2 (A), F102.2
Other:
- note added: "Regulator stability not guaranteed with low ESR output caps"
- note removed: "Warning: regulator stability not guaranteed with low ESR output caps"
- moved on the sheet: C101, C102, C104, C105, C106, D101, F101, J101, R101, U101, U102, U103

Commit message: Tidy up power nets
Other:
- moved on the sheet: D101, R101
Changed lines of the file:
@@
 Wire Wire Line
 	1800 1100 1800 800
-Text HLabel 1000 2700 0    40   BiDi ~ 0
+Text HLabel 1000 2700 0    40   Output ~ 0
 GND
 Wire Wire Line
@@
 $EndComp
 Wire Wire Line
-	2700 1100 2600 1100
+	3400 1100 3300 1100
 $Comp
 L Regulator_Linear:LD1117S33TR_SOT223 U?
@@
 L Device:R R?
 U 1 1 67C00DA5
-P 3400 2250
+P 3300 2250
 AR Path="/67C00DA5" Ref="R?"  Part="1"
 AR Path="/644CBAED/67C00DA5" Ref="R101"  Part="1"
 AR Path="/729F86A7/67C00DA5" Ref="R?"  Part="1"
-F 0 "R101" H 3450 2250 50  0000 L CNN
-F 1 "330R" V 3400 2250 50  0000 C CNN
-F 2 "Resistor_SMD:R_0603_1608Metric_Pad0.98x0.95mm_HandSolder" V 3330 2250 50  0001 C CNN
-F 3 "~" H 3400 2250 50  0001 C CNN
-	1    3400 2250
+F 0 "R101" H 3350 2250 50  0000 L CNN
+F 1 "330R" V 3300 2250 50  0000 C CNN
+F 2 "Resistor_SMD:R_0603_1608Metric_Pad0.98x0.95mm_HandSolder" V 3230 2250 50  0001 C CNN
+F 3 "~" H 3300 2250 50  0001 C CNN
+	1    3300 2250
 	1    0    0    -1
 $EndComp
@@
 	1000 2700 1100 2700
 Wire Wire Line
-	3400 2000 3400 2100
+	3300 2000 3300 2100
 $Comp
 L power:PWR_FLAG #FLG0101
@@
 	1    0    0    -1
 $EndComp
-Wire Wire Line
-	3400 1700 3400 1600
 $Comp
 L Device:LED D?
 U 1 1 67C00D9C
-P 3400 1850
+P 3300 1850
 AR Path="/67C00D9C" Ref="D?"  Part="1"
 AR Path="/644CBAED/67C00D9C" Ref="D101"  Part="1"
 AR Path="/729F86A7/67C00D9C" Ref="D?"  Part="1"
-F 0 "D101" V 3450 1800 50  0000 R CNN
-F 1 "Power" V 3350 1800 50  0000 R CNN
-F 2 "LED_SMD:LED_0603_1608Metric_Pad1.05x0.95mm_HandSolder" H 3400 1850 50  0001 C CNN
-F 3 "~" H 3400 1850 50  0001 C CNN
-	1    3400 1850
+F 0 "D101" V 3350 1800 50  0000 R CNN
+F 1 "Power" V 3250 1800 50  0000 R CNN
+F 2 "LED_SMD:LED_0603_1608Metric_Pad1.05x0.95mm_HandSolder" H 3300 1850 50  0001 C CNN
+F 3 "~" H 3300 1850 50  0001 C CNN
+	1    3300 1850
 	0    -1   -1   0
 $EndComp
-Text HLabel 3400 2500 3    40   BiDi ~ 0
-GND
-Wire Wire Line
-	3400 2400 3400 2500
-Text HLabel 3400 1600 1    40   BiDi ~ 0
-3V3
 Wire Wire Line
 	3700 900  3600 900
-Text HLabel 3700 900  2    40   BiDi ~ 0
+Text HLabel 3700 900  2    40   Output ~ 0
 VUSB
 $Comp
@@
 Wire Wire Line
 	1100 1000 1100 2700
-Text HLabel 2700 1100 2    40   Output ~ 0
+Text HLabel 3400 1100 2    40   Output ~ 0
 3V3
 $Comp
@@
 Wire Wire Line
 	2600 800  2700 800
-Text HLabel 2700 800  2    40   BiDi ~ 0
+Text HLabel 2700 800  2    40   Output ~ 0
 5V
+Wire Wire Line
+	3300 1100 3300 1700
+Connection ~ 3300 1100
+Wire Wire Line
+	3300 1100 2600 1100
+Wire Wire Line
+	3300 2700 3000 2700
+Wire Wire Line
+	3300 2400 3300 2700
+Connection ~ 3000 2700
 $EndSCHEMATC
