File: hardware/HeikouBox/part5-hub.sch (KiCad schematic (older format))
At the start: 51 parts, among them J501 Micro_SD_Card_TFP09-2-12B, J502 RGB, J503 PS/2, Q501 BSS138, Q502 BSS138, Q503 BSS138, SW501 Left, SW502 Up, SW503 Down, SW504 Right, U501 STM32-BluePill-Socket

Commit message: Mainboard v0.1 PCB ready for export
Parts:
- removed J502: RGB, Connector_PinHeader_2.54mm:PinHeader_1x03_P2.54mm_Vertical, symbol Connector_Generic:Conn_01x03
- removed JP501: RGB Bypass, Jumper:SolderJumper-2_P1.3mm_Open_RoundedPad1.0x1.5mm, symbol Jumper:SolderJumper_2_Open
- removed Q501: BSS138, Package_TO_SOT_SMD:SOT-23, symbol Transistor_FET:BSS138
- added R529: 100R, Resistor_SMD:R_0603_1608Metric_Pad0.98x0.95mm_HandSolder, symbol Device:R
- added R530, R531: 1K, Resistor_SMD:R_0603_1608Metric_Pad0.98x0.95mm_HandSolder, symbol Device:R
- R520: value RUSB -> 1K5
- R522: value 1K -> 10K
- R524: value 1K -> 100R
- renumbered C504 to C502, C502 to C503, C503 to C504, SW504 to SW502, SW502 to SW503, SW503 to SW504
Connections:
- net mem_XCAS is gone; now on net MDB5_R: U501.31 (PB3)
- net mem_XCLK is gone; now on net BUTTON_L: U501.13 (PB0)
- net 3V3: now also D501.1 (VDD), D502.1 (VDD), D503.1 (VDD), D504.1 (VDD), R521.1; no longer C501.1, C502.1, C503.1, C504.1, J501.4 (VDD), JP502.1 (A), JP503.3 (B), R509.2, R510.2, R511.2, R512.1, R514.1, R516.1, R518.1, R520.2, R521.2
- net 5V: no longer D501.1 (VDD), D502.1 (VDD), D503.1 (VDD), D504.1 (VDD), R522.2
- net GND: now also R522.2
- net cfg_DONE: now also R531.1; no longer U501.32 (PB4)
- net cfg_NCFG: now also U501.21 (PB12); no longer U501.37 (PB9)
- net cfg_NSTAT: now also R530.1; no longer U501.33 (PB5)
- net SD_SCK: now reaches J501.5 (CLK), U501.10 (PA5)
- net SD_MISO: now reaches J501.7 (DAT0), U501.11 (PA6)
- net SD_MOSI: now reaches J501.3 (CMD), U501.12 (PA7)
- net KEYBOARD_CLK: now reaches Q503.2 (S), R527.1
- net KEYBOARD_CLK: now also U501.7 (PA2); no longer U501.15 (PB10)
- net KEYBOARD_DAT: now reaches Q502.2 (S), R525.1
- net KEYBOARD_DAT: now also U501.6 (PA1); no longer U501.16 (PB11)
- net at U501.2 (PC13): no longer R508.1
- net MDB5_R: now reaches R506.1
- net MDB5_R: no longer U501.21 (PB12)
- net CFG_DONE_R: now reaches U501.23 (PB14)
- net CFG_DONE_R: now also R531.2; no longer R504.1
- net MDB4_CD_R: now reaches R505.1, U501.24 (PB15)
- net MDB2_R: now reaches R503.1
- net MDB2_R: now also U501.27 (PA10); no longer U501.25 (PA8)
- net MDB0_RX_R: now reaches R501.1
- net MDB0_RX_R: now also U501.34 (PB6); no longer U501.26 (PA9)
- net MDB1_TX_R: now reaches R502.1
- net MDB1_TX_R: now also U501.35 (PB7); no longer U501.27 (PA10)
- net USB_DP: now reaches R520.1, U501.29 (PA12)
- net at U501.3 (PC14): no longer R507.1
- net OLED_SCL: now reaches DS501.3 (SCL), R510.1
- net OLED_SCL: now also U501.36 (PB8); no longer U501.34 (PB6)
- net OLED_SDA: now reaches DS501.4 (SDA), R511.1
- net OLED_SDA: now also U501.37 (PB9); no longer U501.35 (PB7)
- net SD_DET: now reaches J501.9 (DET)
- net SD_DET: now also U501.25 (PA8); no longer U501.36 (PB8)
- net BUTTON_L: now reaches C501.2, R513.2
- net BUTTON_L: no longer R512.2, U501.4 (PC15)
- net 3V3_HUB: now reaches U501.40 (3V3)
- net 3V3_HUB: now also C501.1, C502.1, C503.1, C504.1, J501.4 (VDD), JP502.1 (A), JP503.3 (B), R509.1, R510.2, R511.2, R512.2, R514.2, R516.2, R518.2, R520.2
- net NEOPIXEL: now reaches U501.5 (PA0)
- net NEOPIXEL: now also R523.1; no longer R521.1
- net SD_SS: now reaches J501.2 (DAT3/CD), U501.9 (PA4)
- net SD_SS: now also R509.2; no longer R509.1
- net at Q502.3 (D), R526.1: now also R524.1; no longer J503.1
- net at Q503.3 (D), R528.1: now also R529.1; no longer J503.5
- net at D504.2 (DOUT): no longer R524.1
- net at SW503.1: now also R516.1, R517.1; no longer R515.1
- net at SW504.1: now also R518.1, R519.1; no longer R517.1
- net at SW502.1: now also R514.1, R515.1; no longer R519.1
- net at R524.2: now also J503.1
- net PWR_DET: now reaches R522.1
- net PWR_DET: now also R521.2, U501.26 (PA9); no longer R523.1
- net at JP502.2 (C): now also DS501.1 (GND); no longer DS501.2 (VDD)
- net at JP503.2 (C): now also DS501.2 (VDD); no longer DS501.1 (GND)
- net at R513.1, SW501.1: now also R512.1
- net mem_CKE renamed MDB3_R
- net MDB3_R: now also R504.1
- net mem_XWE renamed BUTTON_R
- net BUTTON_R: now also C502.2, R515.2
- new net: J503.5, R529.2
- new net BUTTON_D: C504.2, R519.2, U501.16 (PB11)
- new net BUTTON_U: C503.2, R517.2, U501.15 (PB10)
- new net CFG_NSTAT_R: R530.2, U501.8 (PA3)
- new net MDB6_R: R507.1, U501.32 (PB4)
- new net MDB7_R: R508.1, U501.33 (PB5)
- no-connect marks 9 -> 12
Other:
- note added: "?SPI2_NSS"
- note added: "Core alt functions:\nMDB0 = UART RX?\nMDB1 = UART TX?\nMDB4 = Config DATA0"
- note added: "OLED power pins may be swapped!\nJumpers provided for configuration"
- note added: "Onboard LED"
- note added: "USART1_RX"
- note added: "USART1_TX"
- note added: "USB_DM"
- note added: "WS2812B works okay at 3.3v supply\nThen 3.3v logic needs no shifting"
- note removed: "Gamer RGB go-faster lights"
- note removed: "Keyboard"
- note removed: "Low in both LLHL and LLLH commands, save a pin"
- note removed: "OLED"
- note removed: "PS/2 Clock"
- note removed: "PS/2 Data"
- note removed: "Pulled high to precharge all banks on LLHL command"
- note removed: "RUSB depends on existing pullup on blue pill!\nNone -> RUSB=1K5\n10K -> RUSB=1K8\n4K7 -> RUSB=2K2\n1K5 -> RUSB=None"
- note removed: "SD card"
- note removed: "STM32 Blue Pill"
- note removed: "UART1_RX"
- note removed: "UART1_TX"
- moved on the sheet: C501, C502, C503, C504, D501, D502, D503, D504, DS501, J501, J503, JP502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

Commit message: Tidy up power nets
Other:
- note added: "USB_DM not needed"
- note added: "to resistor fix"
- note removed: "USB_DM"
Changed lines of the file:
@@
 $Descr A4 11693 8268
 encoding utf-8
-Sheet 6 6
+Sheet 5 6
 Title "HeikouBox Mainboard - Hub"
 Date "2021-03-17"
@@
 	3600 1150 3600 1050
 Text Notes 2450 2400 0    40   ~ 0
-USB_DM
+USB_DM not needed
 Wire Wire Line
 	3650 3650 3550 3650
@@
 MDB3_R
 NoConn ~ 2350 2400
-Text Notes 1200 2000 2    40   ~ 0
+Text Notes 1150 2000 2    40   ~ 0
 SPI1_NSS
-Text Notes 1200 2100 2    40   ~ 0
+Text Notes 1150 2100 2    40   ~ 0
 SPI1_SCK
 Text Label 1450 2100 2    40   ~ 0
@@
 Wire Wire Line
 	2450 2900 2350 2900
-Text Notes 2800 3000 0    40   ~ 0
+Text Notes 2850 3050 0    40   ~ 0
 SPI2_SCK
 Wire Wire Line
 	2450 3000 2350 3000
-Text Notes 2800 3100 0    40   ~ 0
+Text Notes 2850 3150 0    40   ~ 0
 ?SPI2_NSS
 Wire Wire Line
@@
 Wire Wire Line
 	1450 2500 1550 2500
-Text Notes 2800 1600 0    40   ~ 0
+Text Notes 2850 1600 0    40   ~ 0
 I2C1_SCL
-Text Notes 2800 1500 0    40   ~ 0
+Text Notes 2850 1500 0    40   ~ 0
 I2C1_SDA
 Wire Wire Line
@@
 NoConn ~ 1550 1300
 Wire Wire Line
-	900  7550 800  7550
-Text HLabel 800  7550 0    40   BiDi ~ 0
+	850  7400 750  7400
+Text HLabel 750  7400 0    40   BiDi ~ 0
 VUSB
 Connection ~ 1550 3100
 Wire Wire Line
 	1550 3100 1550 3000
-Text HLabel 800  7650 0    40   BiDi ~ 0
+Text HLabel 750  7700 0    40   Input ~ 0
 GND
 NoConn ~ 1550 1200
@@
 Connection ~ 9550 5300
 Wire Wire Line
-	2350 1200 2450 1200
-Text Label 2450 1200 0    40   ~ 8
+	2350 1200 2550 1200
+Text Label 2650 1200 0    40   ~ 8
 3V3_HUB
 Text Label 4350 5400 0    40   ~ 8
@@
 	3600 4800 3600 5200
 Wire Wire Line
-	800  7650 900  7650
+	750  7700 850  7700
 Wire Wire Line
 	1550 3100 1450 3100
@@
 Wire Wire Line
 	2350 1300 2450 1300
-Text Label 900  7650 0    40   ~ 8
+Text Label 850  7700 0    40   ~ 8
 GND
-Text Label 900  7550 0    40   ~ 8
+Text Label 850  7400 0    40   ~ 8
 VUSB
 Text Label 3600 1050 1    40   ~ 8
@@
 VUSB
 Wire Wire Line
-	900  7450 800  7450
-Text HLabel 800  7450 0    40   Input ~ 0
+	850  7600 750  7600
+Text HLabel 750  7600 0    40   Input ~ 0
 3V3
-Text Label 900  7450 0    40   ~ 8
+Text Label 850  7600 0    40   ~ 8
 3V3
 Text Label 6500 2200 1    40   ~ 8
@@
 3V3
 Wire Wire Line
-	900  7350 800  7350
-Text HLabel 800  7350 0    40   Input ~ 0
+	850  7500 750  7500
+Text HLabel 750  7500 0    40   Input ~ 0
 5V
-Text Label 900  7350 0    40   ~ 8
+Text Label 850  7500 0    40   ~ 8
 5V
 Text Label 7100 2900 1    40   ~ 8
@@
 Text Label 3400 4100 2    40   ~ 8
 3V3_HUB
+Wire Wire Line
+	2550 1200 2550 1100
+Connection ~ 2550 1200
+Wire Wire Line
+	2550 1200 2650 1200
+$Comp
+L power:PWR_FLAG #FLG0104
+U 1 1 63A8F722
+P 2550 1100
+F 0 "#FLG0104" H 2550 1175 50  0001 C CNN
+F 1 "PWR_FLAG" H 2550 1273 50  0000 C CNN
+F 2 "" H 2550 1100 50  0001 C CNN
+F 3 "~" H 2550 1100 50  0001 C CNN
+	1    2550 1100
+	1    0    0    -1
+$EndComp
+Text Notes 2750 2300 0    40   ~ 0
+to resistor fix
 Wire Bus Line
 	4700 6900 4700 7700
